File: SolderReflowPlate_POWER.kicad_sch (KiCad schematic)
At the start: 21 parts, among them J1 Barrel_Jack_Switch, J3 USB_B_Micro, Q1 WSP4409A, Q2 IRLR8726TRPBF, U1 INA219AIDR, U2 AMS1117-3.3

Commit message: WIP: added LCSC part numbers
Parts:
- removed U2: AMS1117-3.3, Package_TO_SOT_SMD:SOT-223-3_TabPin2, symbol Regulator_Linear:NCP1117-3.3_SOT223
- added D1 (x2): SS54, Diode_SMD:D_SMA, symbol Device:D_Schottky_Filled
- added U5: HT7533-1, Package_TO_SOT_SMD:SOT-89-3, symbol Regulator_Linear:HT75xx-1-SOT89
- C1: value 680uF 16V -> 680uF 35V; LCSC C81137 -> C2980172
- D1: value SS36-E3/57T -> SS54; footprint Diode_SMD:D_SMC -> Diode_SMD:D_SMA; symbol Device:D_Small_Filled -> Device:D_Schottky_Filled; LCSC C35722 -> C22452
- J3: LCSC (none) -> C132350
- Q1: value WSP4409A -> FDS4141-NL-VB; LCSC C2880527 -> C5137404
- R10: footprint Resistor_SMD:R_2010_5025Metric -> Resistor_SMD:R_1206_3216Metric; LCSC C2681035 -> C163046
- R6: LCSC (none) -> C25804
- R6: LCSC (none) -> C23182
Connections:
- net +3V3: now also U5.3 (VOUT)
- net GND: now also U5.1 (GND)
- net VBUS: now also D1.2 (A); no longer C5.1
- net FET_PWM: now reaches Q2.1 (G), R6.1
- net at C19.1, J1.1, Q1.5 (D)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: now also D1.2 (A)
- new net: C5.1, D1.1 (K), D1.1 (K), U5.2 (VIN)
Other:
- note added: "AMS1117-3.3 1A output, 15V absmax HT7533-1 100mA output, 30V absmax"
- moved on the sheet: C19, C5, C7
